Commit message: did some changes in collision part of the robot.urdf file

File: robot.urdf (robot description, URDF)
Before this commit: robot differential_drive_robot, 1 links, 0 joints
Links:
- link base_link: geometry collision box size=0.20 0.15 0.06; visual mesh filename=package://assets/base_link.stl

Commit message: did some crazy changes

File: robot.urdf (robot description, URDF)
Before this commit: robot differential_drive_robot, 1 links, 0 joints
Links:
- added link base_footprint
- added link caster_wheel, mass 0.1; collision sphere radius=0.015; visual sphere radius=0.015
- added link left_wheel, mass 0.2; collision cylinder length=0.025 radius=0.033; visual cylinder length=0.025 radius=0.033
- added link right_wheel, mass 0.2; collision cylinder length=0.025 radius=0.033; visual cylinder length=0.025 radius=0.033
- link base_link: mass 0.731356 -> 0.8; geometry collision box size=0.2 0.15 0.06; visual box size=0.2 0.15 0.06
Joints:
- added joint base_joint: type fixed, parent base_footprint, child base_link, origin xyz=0 0 0.033 rpy=0 0 0
- added joint caster_joint: type fixed, parent base_link, child caster_wheel, origin xyz=0.08 0 -0.018 rpy=0 0 0
- added joint left_wheel_joint: type continuous, parent base_link, child left_wheel, origin xyz=0 0.09 0 rpy=0 0 0, axis 0 1 0
- added joint right_wheel_joint: type continuous, parent base_link, child right_wheel, origin xyz=0 -0.09 0 rpy=0 0 0, axis 0 1 0

Commit message: Added some libraries for slam navigation in the container

File: robot.urdf (robot description, URDF)
Before this commit: robot tushar_car, 5 links, 4 joints
Links:
- link base_link: mass 0.8 -> 0.5
- link caster_wheel: mass 0.1 -> 0.05
- link left_wheel: mass 0.2 -> 0.1
- link right_wheel: mass 0.2 -> 0.1

Commit message: Added some crazy things

File: robot.urdf (robot description, URDF)
Before this commit: robot tushar_car, 5 links, 4 joints
Links:
- removed link base_footprint
- added link laser_frame, mass 0.1; collision cylinder length=0.04 radius=0.05; visual cylinder length=0.04 radius=0.05
- link base_link: mass 0.5 -> 5.0; geometry collision box size=0.5 0.3 0.15; visual box size=0.5 0.3 0.15
- link caster_wheel: mass 0.05 -> 0.2; geometry collision sphere radius=0.05; visual sphere radius=0.05
- link left_wheel: mass 0.1 -> 0.5; geometry collision cylinder length=0.05 radius=0.1; visual cylinder length=0.05 radius=0.1
- link right_wheel: mass 0.1 -> 0.5; geometry collision cylinder length=0.05 radius=0.1; visual cylinder length=0.05 radius=0.1
Joints:
- removed joint base_joint
- removed joint caster_joint
- added joint caster_wheel_joint: type fixed, parent base_link, child caster_wheel, origin xyz=0.15 0 -0.1 rpy=0 0 0
- added joint laser_joint: type fixed, parent base_link, child laser_frame, origin xyz=0.1 0 0.095 rpy=0 0 0
- joint left_wheel_joint: axis 0 1 0 -> 0 0 1; origin xyz=0 0.09 0 rpy=0 0 0 -> xyz=-0.1 0.175 -0.05 rpy=-1.5708 0 0
- joint right_wheel_joint: axis 0 1 0 -> 0 0 1; origin xyz=0 -0.09 0 rpy=0 0 0 -> xyz=-0.1 -0.175 -0.05 rpy=-1.5708 0 0
